Commit message: till gazebo

File: robot_description/urdf/opensg_robot.gazebo.mesh.xacro (robot description, xacro)
@@ -88,5 +88,5 @@
   <gazebo reference="front_base_scan">
     <material>Gazebo/FlatBlack</material>
-    <sensor type="ray" name="lds_lfcd_sensor">
+    <sensor type="ray" name="lds_lfcd_sensor_1">
       <pose>0 0 0 0 0 0</pose>
       <visualize>$(arg laser_visual)</visualize>
@@ -97,12 +97,14 @@
             <samples>360</samples>
             <resolution>1</resolution>
-            <min_angle>-3.00</min_angle> -3.14 / 0.00
-            <max_angle>1.57</max_angle>  1.57 / 6.28139
+            <!-- <min_angle>-1.85</min_angle> -->
+            <min_angle>-1.5707</min_angle>
+            <!-- <max_angle>1.85</max_angle> -->
+            <max_angle>1.5707</max_angle>
           </horizontal>
         </scan>
         <range>
-          <min>0.3</min> 0.30
-          <max>7.5</max> 10.0
-          <resolution>0.015</resolution> 0.015
+          <min>0.120</min>
+          <max>3.5</max>
+          <resolution>0.015</resolution>
         </range>
         <noise>
@@ -118,9 +120,9 @@
     </sensor>
   </gazebo>
-  <!-- <gazebo reference="rear_base_scan">
+  <gazebo reference="rear_base_scan">
     <material>Gazebo/FlatBlack</material>
-    <sensor type="ray" name="lds_lfcd_sensor">
+    <sensor type="ray" name="lds_lfcd_sensor_2">
       <pose>0 0 0 0 0 0</pose>
-      <visualize>$(arg laser_visual_2)</visualize>
+      <visualize>$(arg laser_visual)</visualize>
       <update_rate>5</update_rate>
       <ray>
@@ -129,6 +131,8 @@
             <samples>360</samples>
             <resolution>1</resolution>
-            <min_angle>2.80</min_angle> 0.00
-            <max_angle>-1.30</max_angle>  6.28139
+            <!-- <min_angle>-1.85</min_angle> -->
+            <min_angle>-1.5707</min_angle>
+            <!-- <max_angle>1.85</max_angle> -->
+            <max_angle>1.5707</max_angle>
           </horizontal>
         </scan>
@@ -136,5 +140,5 @@
           <min>0.120</min>
           <max>3.5</max>
-          <resolution>0.015</resolution> 0.015
+          <resolution>0.015</resolution>
         </range>
         <noise>
@@ -146,7 +150,7 @@
       <plugin name="gazebo_ros_lds_lfcd_controller" filename="libgazebo_ros_laser.so">
         <topicName>opensg_scan_rear</topicName>
-        <frameName>base_footprint</frameName>
+        <frameName>rear_base_scan</frameName>
       </plugin>
     </sensor>
-  </gazebo> -->
+  </gazebo>
 </robot>

File: robot_description/urdf/opensg_robot.gazebo.xacro (robot description, xacro)
@@ -70,7 +70,7 @@
     </plugin>
   </gazebo>
-  <gazebo reference="base_scan">
+  <gazebo reference="front_base_scan">
     <material>Gazebo/FlatBlack</material>
-    <sensor type="ray" name="lds_lfcd_sensor">
+    <sensor type="ray" name="lds_lfcd_sensor_1">
       <pose>0 0 0 0 0 0</pose>
       <visualize>$(arg laser_visual)</visualize>
@@ -81,6 +81,6 @@
             <samples>360</samples>
             <resolution>1</resolution>
-            <min_angle>-1.85</min_angle> 0.00
-            <max_angle>1.85</max_angle>  6.28139
+            <min_angle>-1.85</min_angle>
+            <max_angle>1.85</max_angle>
           </horizontal>
         </scan>
@@ -88,5 +88,5 @@
           <min>0.120</min>
           <max>3.5</max>
-          <resolution>0.015</resolution> 0.015
+          <resolution>0.015</resolution>
         </range>
         <noise>
@@ -98,5 +98,37 @@
       <plugin name="gazebo_ros_lds_lfcd_controller" filename="libgazebo_ros_laser.so">
         <topicName>opensg_scan_front</topicName>
-        <frameName>base_footprint</frameName>
+        <frameName>front_base_scan</frameName>
+      </plugin>
+    </sensor>
+  </gazebo>
+  <gazebo reference="rear_base_scan">
+    <material>Gazebo/FlatBlack</material>
+    <sensor type="ray" name="lds_lfcd_sensor_2">
+      <pose>0 0 0 0 0 0</pose>
+      <visualize>$(arg laser_visual)</visualize>
+      <update_rate>5</update_rate>
+      <ray>
+        <scan>
+          <horizontal>
+            <samples>360</samples>
+            <resolution>1</resolution>
+            <min_angle>-1.85</min_angle>
+            <max_angle>1.85</max_angle>
+          </horizontal>
+        </scan>
+        <range>
+          <min>0.120</min>
+          <max>3.5</max>
+          <resolution>0.015</resolution>
+        </range>
+        <noise>
+          <type>gaussian</type>
+          <mean>0.0</mean>
+          <stddev>0.01</stddev>
+        </noise>
+      </ray>
+      <plugin name="gazebo_ros_lds_lfcd_controller" filename="libgazebo_ros_laser.so">
+        <topicName>opensg_scan_rear</topicName>
+        <frameName>rear_base_scan</frameName>
       </plugin>
     </sensor>

File: robot_description/urdf/opensg_robot.urdf.mesh.xacro (robot description, xacro)
@@ -168,5 +168,5 @@
     <parent link="base_link"/>
     <child link="rear_base_scan"/>
-    <origin xyz="-0.545 0.370 0.195" rpy="0 0 0"/>
+    <origin xyz="-0.545 0.370 0.195" rpy="0 0 3.1415"/>
   </joint>
   <link name="rear_base_scan">
